File: Loom.kicad_sch (KiCad schematic)
At the start: 53 parts

Commit message: Update post-FSUK '25
Parts:
- SPKC1: value Bosch Jetronic -> Junior Power Timer; symbol Connector_Generic:Conn_01x04 -> Connector_Generic:Conn_01x05
- SPKC2: symbol Connector_Generic:Conn_01x05 -> Connector_Generic:Conn_01x04
Connections:
- net GND: now also SPKC1.3 (Pin_3); no longer SPKC2.3 (Pin_3)
- net SPKA: now also SPKC1.5 (Pin_5); no longer SPKC1.4 (Pin_4)
- net SPKB: now also SPKC1.4 (Pin_4); no longer SPKC1.3 (Pin_3)
- net at SPK3.2 (Pin_2): now also SPKC2.3 (Pin_3); no longer SPKC2.4 (Pin_4)
- net at SPK4.2 (Pin_2): now also SPKC2.4 (Pin_4); no longer SPKC2.5 (Pin_5)
Other:
- note added: "Base 1 Base 2 Base 3 Base 4"
- note added: "Coll 1 Coll 2 Ground Coll 3 Coll 4"
- note added: "Currently botched to connect to SEN5V"
- note added: "Currently botched to connect to SENGND"
- note removed: "Base 1 Base 2 Gnd Base 3 Base 4"
- note removed: "Coll 1 Coll 2 Coll 3 Coll 4"
- note removed: "ECU 2A Lambda 5A Stepper 5A Misc 10A INJA 5A INJB 5A FP 10A SPK 20A Fan 20A"
Changed lines of the file:
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@@
 		)
 	)
-	(text "ECU  2A\nLambda  5A\nStepper  5A\nMisc 10A\n\nINJA  5A\nINJB  5A\nFP 10A\nSPK 20A\nFan 20A\n "
-		(exclude_from_sim no)
-		(at 637.54 281.94 0)
-		(effects
-			(font
-				(size 1.5748 1.5748)
-			)
-			(justify right)
-		)
-	)
 	(text "ECU 2A\nLambda 5A\nETC CU 5A\nETC Stepper 5A\nShutdown 5A\nQS CU 5A\nBrake Light 5A\nMisc 10A\n\n\n\nINJA 5A\nINJB 5A\nFP 10A\nSpark 20A\nFans 20A\n "
 		(exclude_from_sim no)
@@
 		)
 	)
+	(text "Currently botched to connect to SEN5V"
+		(exclude_from_sim no)
+		(at 144.78 25.4 0)
+		(effects
+			(font
+				(size 1.27 1.27)
+			)
+			(justify left bottom)
+		)
+	)
 	(text "Gnd\nSolenoid Up\nSolenoid Dn"
 		(exclude_from_sim no)
@@
 		)
 	)
+	(text "Currently botched to connect to SENGND"
+		(exclude_from_sim no)
+		(at 144.78 30.48 0)
+		(effects
+			(font
+				(size 1.27 1.27)
+			)
+			(justify left bottom)
+		)
+	)
 	(text "FIREWALL CONNECTOR\nHDP24-24-31SE\n\nPinout:\n 1 MiscPWR\n 2 ETC CU Power\n 3 StepperPWR\n 4 IdleCtrl\n 5 Blip\n 6 TPS Power 1\n 7 TPS Signal 1\n 8 TPS Ground 1\n 9 TPS Power 2\n10 TPS Signal 2\n11 TPS Ground 2\n12 Stepper 1+\n13 Stepper 1-\n14 Stepper 2+\n15 Stepper 2-\n16 Neutral\n17 Shift Down\n18 Shift Up\n19 Tachometer\n20 Shutdown Out\n21 Starter Sig\n22 Fan Sig\n23 BLS Sig\n24 Launch Sig\n25 Launch LED\n26 \n27 \n28 Brake Light PWR\n29 CANH\n30 CANL\n31 Shutdown PWR"
 		(exclude_from_sim no)
@@
 		)
 	)
-	(text "Base 1\nBase 2\nGnd\nBase 3\nBase 4"
+	(text "Base 1\nBase 2\nBase 3\nBase 4\n "
 		(exclude_from_sim no)
 		(at 523.24 45.72 0)
@@
 		)
 	)
-	(text "Coll 1\nColl 2\nColl 3\nColl 4\n "
+	(text "Coll 1\nColl 2\nGround\nColl 3\nColl 4"
 		(exclude_from_sim no)
 		(at 502.92 45.72 0)
@@
 	)
 	(junction
+		(at 487.68 40.64)
+		(diameter 0)
+		(color 0 0 0 0)
+	)
+	(junction
 		(at 403.86 38.1)
 		(diameter 0)
@@
 	)
 	(junction
+		(at 490.22 43.18)
+		(diameter 0)
+		(color 0 0 0 0)
+	)
+	(junction
 		(at 533.4 307.34)
 		(diameter 0)
@@
 	)
 	(junction
-		(at 490.22 40.64)
-		(diameter 0)
-		(color 0 0 0 0)
-	)
-	(junction
 		(at 538.48 25.4)
 		(diameter 0)
@@
 	)
 	(junction
-		(at 492.76 43.18)
-		(diameter 0)
-		(color 0 0 0 0)
-	)
-	(junction
 		(at 558.8 167.64)
 		(diameter 0)
@@
 	(wire
 		(pts
-			(xy 530.86 50.8) (xy 530.86 66.04)
-		)
-		(stroke
-			(width 0)
-			(type default)
-		)
-	)
-	(wire
-		(pts
 			(xy 469.9 86.36) (xy 528.32 86.36)
 		)
@@
 	(wire
 		(pts
+			(xy 492.76 45.72) (xy 495.3 45.72)
+		)
+		(stroke
+			(width 0)
+			(type default)
+		)
+	)
+	(wire
+		(pts
 			(xy 289.56 177.8) (xy 373.38 177.8)
 		)
@@
 	(wire
 		(pts
-			(xy 535.94 45.72) (xy 535.94 71.12)
-		)
-		(stroke
-			(width 0)
-			(type default)
-		)
-	)
-	(wire
-		(pts
-			(xy 533.4 48.26) (xy 533.4 53.34)
+			(xy 533.4 45.72) (xy 533.4 53.34)
 		)
 		(stroke
@@
 	(wire
 		(pts
-			(xy 490.22 48.26) (xy 490.22 40.64)
+			(xy 487.68 40.64) (xy 487.68 50.8)
 		)
 		(stroke
@@
 	(wire
 		(pts
-			(xy 439.42 40.64) (xy 490.22 40.64)
+			(xy 439.42 40.64) (xy 487.68 40.64)
 		)
 		(stroke
@@
 	(wire
 		(pts
-			(xy 492.76 43.18) (xy 492.76 45.72)
+			(xy 210.82 228.6) (xy 243.84 228.6)
 		)
 		(stroke
@@
 	(wire
 		(pts
-			(xy 210.82 228.6) (xy 243.84 228.6)
+			(xy 525.78 162.56) (xy 525.78 292.1)
 		)
 		(stroke
 			(width 0)
 			(type default)
+			(color 255 0 0 1)
 		)
 	)
 	(wire
 		(pts
-			(xy 525.78 162.56) (xy 525.78 292.1)
+			(xy 538.48 25.4) (xy 538.48 22.86)
 		)
 		(stroke
@@
 	(wire
 		(pts
-			(xy 538.48 25.4) (xy 538.48 22.86)
+			(xy 530.86 45.72) (xy 533.4 45.72)
 		)
 		(stroke
 			(width 0)
 			(type default)
-			(color 255 0 0 1)
 		)
 	)
 	(wire
 		(pts
-			(xy 530.86 48.26) (xy 533.4 48.26)
+			(xy 490.22 43.18) (xy 490.22 48.26)
 		)
 		(stroke
@@
 	(wire
 		(pts
+			(xy 530.86 48.26) (xy 530.86 66.04)
+		)
+		(stroke
+			(width 0)
+			(type default)
+		)
+	)
+	(wire
+		(pts
 			(xy 157.48 248.92) (xy 38.1 248.92)
 		)
@@
 	(wire
 		(pts
-			(xy 441.96 43.18) (xy 492.76 43.18)
+			(xy 441.96 43.18) (xy 490.22 43.18)
 		)
 		(stroke
@@
 	(wire
 		(pts
+			(xy 492.76 55.88) (xy 492.76 45.72)
+		)
+		(stroke
+			(width 0)
+			(type default)
+		)
+	)
+	(wire
+		(pts
 			(xy 546.1 50.8) (xy 538.48 50.8)
 		)
@@
 	(wire
 		(pts
-			(xy 495.3 48.26) (xy 490.22 48.26)
+			(xy 495.3 50.8) (xy 487.68 50.8)
 		)
 		(stroke
@@
 	(wire
 		(pts
-			(xy 492.76 45.72) (xy 495.3 45.72)
+			(xy 490.22 48.26) (xy 495.3 48.26)
 		)
 		(stroke
@@
 	(wire
 		(pts
+			(xy 487.68 40.64) (xy 495.3 40.64)
+		)
+		(stroke
+			(width 0)
+			(type default)
+		)
+	)
+	(wire
+		(pts
 			(xy 543.56 127) (xy 543.56 129.54)
 		)
@@
 	(wire
 		(pts
+			(xy 490.22 43.18) (xy 495.3 43.18)
+		)
+		(stroke
+			(width 0)
+			(type default)
+		)
+	)
+	(wire
+		(pts
 			(xy 457.2 208.28) (xy 462.28 208.28)
 		)
@@
 	(wire
 		(pts
-			(xy 530.86 45.72) (xy 535.94 45.72)
-		)
-		(stroke
-			(width 0)
-			(type default)
-		)
-	)
-	(wire
-		(pts
 			(xy 203.2 35.56) (xy 142.24 35.56)
 		)
@@
 	(wire
 		(pts
-			(xy 495.3 43.18) (xy 492.76 43.18)
-		)
-		(stroke
-			(width 0)
-			(type default)
-		)
-	)
-	(wire
-		(pts
 			(xy 142.24 289.56) (xy 142.24 340.36)
 		)
@@
 	(wire
 		(pts
-			(xy 490.22 40.64) (xy 495.3 40.64)
-		)
-		(stroke
-			(width 0)
-			(type default)
-		)
-	)
-	(wire
-		(pts
 			(xy 406.4 66.04) (xy 396.24 66.04)
 		)
@@
 	(symbol
 		(lib_id "power:GND")
-		(at 535.94 71.12 0)
+		(at 492.76 55.88 0)
 		(unit 1)
 		(exclude_from_sim no)
@@
 		(fields_autoplaced yes)
 		(property "Reference" "#PWR01"
-			(at 535.94 77.47 0)
+			(at 492.76 62.23 0)
 			(effects
 				(font
@@
 		)
 		(property "Value" "GND"
-			(at 535.94 76.2 0)
+			(at 492.76 60.96 0)
 			(effects
 				(font
@@
 		)
 		(property "Footprint" ""
-			(at 535.94 71.12 0)
+			(at 492.76 55.88 0)
 			(effects
 				(font
@@
 		)
 		(property "Datasheet" ""
-			(at 535.94 71.12 0)
+			(at 492.76 55.88 0)
 			(effects
 				(font
@@
 		)
 		(property "Description" "Power symbol creates a global label with name \"GND\" , ground"
-			(at 535.94 71.12 0)
+			(at 492.76 55.88 0)
 			(effects
 				(font
@@
 	)
 	(symbol
-		(lib_id "Connector_Generic:Conn_01x05")
-		(at 525.78 45.72 0)
+		(lib_id "Connector_Generic:Conn_01x04")
+		(at 525.78 43.18 0)
 		(mirror y)
 		(unit 1)
@@
 		(dnp no)
 		(property "Reference" "SPKC2"
-			(at 528.32 35.56 0)
+			(at 528.32 33.02 0)
 			(effects
 				(font
@@
 		)
 		(property "Value" "Bosch Jetronic"
-			(at 528.32 38.1 0)
+			(at 528.32 35.56 0)
 			(effects
 				(font
@@
 				)
 				(justify left)
+				(hide yes)
 			)
 		)
 		(property "Footprint" ""
-			(at 525.78 45.72 0)
+			(at 525.78 43.18 0)
 			(effects
 				(font
@@
 		)
 		(property "Datasheet" "~"
-			(at 525.78 45.72 0)
+			(at 525.78 43.18 0)
 			(effects
 				(font
@@
 			)
 		)
-		(property "Description" "Generic connector, single row, 01x05, script generated (kicad-library-utils/schlib/autogen/connector/)"
-			(at 525.78 45.72 0)
+		(property "Description" "Generic connector, single row, 01x04, script generated (kicad-library-utils/schlib/autogen/connector/)"
+			(at 525.78 43.18 0)
 			(effects
 				(font
@@
 		(pin "4"
 		)
-		(pin "5"
-		)
 		(instances
 			(project ""
@@
 	)
 	(symbol
-		(lib_id "Connector_Generic:Conn_01x04")
-		(at 500.38 43.18 0)
+		(lib_id "Connector_Generic:Conn_01x05")
+		(at 500.38 45.72 0)
 		(unit 1)
 		(exclude_from_sim no)
@@
 			)
 		)
-		(property "Value" "Bosch Jetronic"
-			(at 497.84 38.1 0)
+		(property "Value" "Junior Power Timer"
+			(at 502.92 38.1 0)
 			(effects
 				(font
@@
 		)
 		(property "Footprint" ""
-			(at 500.38 43.18 0)
+			(at 500.38 45.72 0)
 			(effects
 				(font
@@
 		)
 		(property "Datasheet" "~"
-			(at 500.38 43.18 0)
+			(at 500.38 45.72 0)
 			(effects
 				(font
@@
 			)
 		)
-		(property "Description" "Generic connector, single row, 01x04, script generated (kicad-library-utils/schlib/autogen/connector/)"
-			(at 500.38 43.18 0)
+		(property "Description" "Generic connector, single row, 01x05, script generated (kicad-library-utils/schlib/autogen/connector/)"
+			(at 500.38 45.72 0)
 			(effects
 				(font
@@
 		(pin "4"
 		)
+		(pin "5"
+		)
 		(instances
